File: Hardware/PCB/Eagle/Jacdac_Proto_Board.brd (EAGLE design)
At the start: 54.9 x 38.1 mm, 14 parts, among them SW1 CUI_SJ1-3513, SW2 CUI_SJ1-3513

Commit message: Updated PCB design files
Parts:
- added U$2: MILADOR-LOGO-, milador:MILADOR_LOGO1
Other:
- board text added: "Jacdac-Proto-Board"
Changed lines of the file:
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@@
 <drawing>
 <settings>
-<setting alwaysvectorfont="no"/>
+<setting alwaysvectorfont="yes"/>
 <setting keepoldvectorfont="yes"/>
 <setting verticaltext="up"/>
@@
 <circle x="2.54" y="14.224" radius="0.254" width="0.508" layer="22"/>
 <circle x="40.64" y="23.876" radius="0.254" width="0.508" layer="22"/>
+<text x="23.622" y="23.876" size="1.27" layer="22" ratio="20" rot="MR0">Jacdac-Proto-Board</text>
 </plain>
 <attributes>
@@
 <attribute name="VALUE" x="3.81" y="24.892" size="0.6096" layer="27" font="vector" ratio="20"/>
 </element>
+<element name="U$2" library="milador" library_urn="urn:adsk.eagle:library:12595918" package="MILADOR_LOGO1" package3d_urn="urn:adsk.eagle:package:28431737/1" value="MILADOR-LOGO-" x="30.734" y="23.622" smashed="yes" rot="MR0"/>
 </elements>
 <signals>
@@
 </signals>
 <mfgpreviewcolors>
-<mfgpreviewcolor name="soldermaskcolor" color="0xC8AA0000"/>
+<mfgpreviewcolor name="soldermaskcolor" color="0xC8009100"/>
 <mfgpreviewcolor name="silkscreencolor" color="0xFFFEFEFE"/>
 <mfgpreviewcolor name="backgroundcolor" color="0xFF282828"/>
