File: Hardware/PCB/Eagle/Jacdac_Proto_Board.sch (EAGLE design)
At the start: 14 parts, among them SW1 CUI_SJ1-3513, SW2 CUI_SJ1-3513

Commit message: Updated PCB design files
Parts:
- added U$2: MILADOR-LOGO-, milador:MILADOR-LOGO-
Changed lines of the file:
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@@
 <part name="J6" library="milador" library_urn="urn:adsk.eagle:library:12595918" deviceset="CONNECTORS_CONN_01" device="PTH_NO_SILK_YES_STOP" package3d_urn="urn:adsk.eagle:package:29222250/2"/>
 <part name="FRAME1" library="frames" library_urn="urn:adsk.eagle:library:229" deviceset="A4L-LOC" device=""/>
+<part name="U$2" library="milador" library_urn="urn:adsk.eagle:library:12595918" deviceset="MILADOR-LOGO-" device="" package3d_urn="urn:adsk.eagle:package:28431737/1"/>
 </parts>
 <sheets>
@@
 <attribute name="SHEET" x="230.505" y="5.08" size="2.54" layer="94"/>
 </instance>
+<instance part="U$2" gate="G$1" x="149.86" y="45.72" smashed="yes"/>
 </instances>
 <busses>
